File: Audio_DAC_addon.sch (KiCad schematic (older format))
At the start: 8 parts, among them J16 Conn_01x10, J17 Conn_01x08, J25 Conn_01x10, J28 Conn_01x10, J29 Conn_01x01

Commit message: real initial commit
Parts:
- added C10, C4, C5, C7, C8, C9: 1uF, Capacitors_SMD:C_0402_NoSilk, symbol C
- added C6: 2.2uF, Capacitors_SMD:C_0402_NoSilk, symbol C
- added J1: Audio-Jack-3, custom:AUB-11_audio-jack, symbol Audio-Jack-3
- added R1, R2, R3, R4: R, Resistors_SMD:R_0603_HandSoldering, symbol R
- added U1: MAX9860, Housings_DFN_QFN:QFN-24-1EP_4x4mm_Pitch0.5mm, symbol MAX9860
Connections:
- net labels added: BCLK, DVDD, DVDDIO_3V3, LRCLK, MCLK, SDIN
- wire segments 36 -> 90

Commit message: add LDOs + pcb progress
Parts:
- added C11, C12, C13, C14, C15, C16: 1uF, Capacitors_SMD:C_0402_NoSilk, symbol C
- added U2: TLV70033DCKR, TO_SOT_Packages_SMD:SOT-23-5, symbol TLV70033DCKR
- added U3, U4: TLV70018DDCR, TO_SOT_Packages_SMD:SOT-23-5, symbol TLV70018DDCR
Connections:
- net labels added: AVDD, IRQ
- wire segments 90 -> 114
Other:
- moved on the sheet: J29

Commit message: pcb and circuit diagram are almost done
Parts:
- removed C1, C2, C3: 0.1, Capacitors_SMD:C_0402_NoSilk, symbol C
- removed J17: Conn_01x08, Pin_Headers:Pin_Header_Straight_1x08_Pitch2.54mm, symbol Conn_01x08
- removed J29: Conn_01x01, Mounting_Holes:MountingHole_3.2mm_M3_ISO7380_Pad, symbol Conn_01x01
- added J2: Conn_01x03, Pin_Headers:Pin_Header_Straight_1x03_Pitch2.54mm, symbol Conn_01x03
- added R10, R11, R5, R6, R7, R8, R9: R, Resistors_SMD:R_0603_HandSoldering, symbol R
Connections:
- net labels added: FPGA_AE15, FPGA_AF17, OUTN, OUTP, SCL, SDA
- net labels removed: FPGA_AF13, FPGA_AG10, FPGA_AG13
- wire segments 114 -> 116
Other:
- moved on the sheet: C10, C11, C12, C13, C14, C15, C16, C4, C5, C6, C7, C8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

Commit message: generate gerber + lots of bug fix
Connections:
- net labels added: MICBIAS, PREG, REF, REG
Changed lines of the file:
@@
 	8500 2100 8500 2450
 Connection ~ 8500 2300
-Text Label 9000 2750 0    60   ~ 0
+Text Label 8300 2750 0    60   ~ 0
 AVDD
 Text Label 6450 2450 0    60   ~ 0
@@
 Text Label 2800 2400 0    60   ~ 0
 FPGA_AF17
+Text Label 8300 2850 0    60   ~ 0
+MICBIAS
+Text Label 8300 2950 0    60   ~ 0
+REG
+Text Label 8300 3050 0    60   ~ 0
+PREG
+Text Label 8300 3150 0    60   ~ 0
+REF
 $EndSCHEMATC
